File: hardware/.portability/backup/comanda_pompa_ A0121A4.kicad_sch (KiCad schematic)
At the start: 41 parts, among them J10 RS485_M, J11 NC (test led), J2 220V IN, J4 BUTON Power, J5 NC (test led), J6 CONSOLA, J7 LEDS, J8 LED, J9 RS485_uC, Q2 BD139, T1 Transformer_1P_1S, U1 ATmega328P-P, U2 XL4015, U3 4N25, U4 ULN2003, Y1 16MHz

Commit message: module in hardware
Parts:
- U2: value XL4015 -> XL4016_ADJ
Other:
- note removed: "https://www.drot.ro/platforma-arduino/121946-modul-step-down-4a-xl4015-dc-dc-cc-cv.html"
Changed lines of the file:
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@@
 		)
 	)
-	(text "https://www.drot.ro/platforma-arduino/121946-modul-step-down-4a-xl4015-dc-dc-cc-cv.html"
-		(exclude_from_sim no)
-		(at 94.742 184.912 0)
-		(effects
-			(font
-				(size 1.27 1.27)
-			)
-		)
-	)
 	(text "MIJLOC"
 		(exclude_from_sim no)
@@
 			)
 		)
-		(property "Value" "XL4015"
+		(property "Value" "XL4016_ADJ"
 			(at 101.6 154.94 0)
 			(show_name no)
